File: Extra_Sheet.kicad_sch (KiCad schematic)
At the start: 9 parts, among them J6 ST, K1 SANYOU_SRD_Form_C, Q1 BC817

Commit message: PCB Components placed
Parts:
- added H1, H2, H3, H4: MountingHole_Pad, MountingHole:MountingHole_3.2mm_M3_Pad_Via, symbol Mechanical:MountingHole_Pad

Commit message: pcb finished, gerber added
Connections:
- net Relay_Ctrl: now reaches R6.1
- no-connect marks 0 -> 4
Changed lines of the file:
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@@
 		(color 0 0 0 0)
 	)
+	(no_connect
+		(at 224.79 92.71)
+	)
+	(no_connect
+		(at 224.79 82.55)
+	)
+	(no_connect
+		(at 224.79 87.63)
+	)
+	(no_connect
+		(at 224.79 97.79)
+	)
 	(wire
 		(pts
@@
 		(pts
 			(xy 143.51 100.33) (xy 143.51 101.6)
+		)
+		(stroke
+			(width 0)
+			(type default)
+		)
+	)
+	(wire
+		(pts
+			(xy 119.38 106.68) (xy 124.46 106.68)
 		)
 		(stroke
@@
 			)
 		)
+	)
+	(global_label "Relay_Ctrl"
+		(shape input)
+		(at 119.38 106.68 180)
+		(fields_autoplaced yes)
+		(effects
+			(font
+				(size 1.27 1.27)
+			)
+			(justify right)
+		)
+		(property "Intersheetrefs" "${INTERSHEET_REFS}"
+			(at 106.8397 106.68 0)
+			(effects
+				(font
+					(size 1.27 1.27)
+				)
+				(justify right)
+				(hide yes)
+			)
+		)
