File: STM32_base.kicad_sch (KiCad schematic)
At the start: 34 parts, among them J1 TC2030-NL, J2 Conn_01x04_Pin, J3 ST, J4 Conn_01x04_Pin, J5 USB_C_Receptacle_USB2.0_14P, SW1 SW_Push, U1 STM32F103C8Tx, U2 USBLC6-2P6, U3 AMS1117-3.3, Y1 8MHz

Commit message: PCB Components placed
Parts:
- removed L1: 1mH, Inductor_THT:L_CommonMode_Wuerth_WE-CMB-M, symbol Device:L_Coupled_1324
- added FL1: Choke_Schaffner_RN102-2-02-1M1, Inductor_THT:Choke_Schaffner_RN102-04-14.0x14.0mm, symbol Filter:Choke_Schaffner_RN102-2-02-1M1
- C11: footprint Capacitor_THT:CP_Radial_D7.5mm_P2.50mm -> Capacitor_SMD:CP_Elec_10x10
Connections:
- net LINE-OUT: now also FL1.2
- net NEUT: now also FL1.3
- net NEUT-OUT: now also FL1.4
- net at C9.1, RV1.1, TH1.1: now also FL1.1
Other:
- sheet Extra Sheet renamed Relay & Mountint Holes
Changed lines of the file:
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@@
 			)
 		)
-		(property "Footprint" "Capacitor_THT:CP_Radial_D7.5mm_P2.50mm"
+		(property "Footprint" "Capacitor_SMD:CP_Elec_10x10"
 			(at 156.21 44.45 0)
 			(effects
@@
 	)
 	(symbol
-		(lib_id "Device:L_Coupled_1324")
-		(at 93.98 44.45 0)
-		(unit 1)
-		(exclude_from_sim no)
-		(in_bom yes)
-		(on_board yes)
-		(dnp no)
-		(fields_autoplaced yes)
-		(property "Reference" "L1"
-			(at 93.599 36.83 0)
-			(effects
-				(font
-					(size 1.27 1.27)
-				)
-			)
-		)
-		(property "Value" "1mH"
-			(at 93.599 39.37 0)
-			(effects
-				(font
-					(size 1.27 1.27)
-				)
-			)
-		)
-		(property "Footprint" "Inductor_THT:L_CommonMode_Wuerth_WE-CMB-M"
-			(at 93.98 44.45 0)
-			(effects
-				(font
-					(size 1.27 1.27)
-				)
-				(hide yes)
-			)
-		)
-		(property "Datasheet" "~"
-			(at 93.98 44.45 0)
-			(effects
-				(font
-					(size 1.27 1.27)
-				)
-				(hide yes)
-			)
-		)
-		(property "Description" "Coupled inductor"
-			(at 93.98 44.45 0)
-			(effects
-				(font
-					(size 1.27 1.27)
-				)
-				(hide yes)
-			)
-		)
-		(pin "3"
-		)
-		(pin "2"
-		)
-		(pin "1"
-		)
-		(pin "4"
-		)
-		(instances
-			(project "STM32_base"
-				(path "/9959bbda-b5da-43e8-8c0f-a51c8fc16f77"
-					(reference "L1")
-					(unit 1)
-				)
-			)
-		)
-	)
-	(symbol
 		(lib_id "Connector:Conn_ARM_SWD_TagConnect_TC2030-NL")
 		(at 139.7 110.49 0)
@@
 				(path "/9959bbda-b5da-43e8-8c0f-a51c8fc16f77"
 					(reference "R2")
+					(unit 1)
+				)
+			)
+		)
+	)
+	(symbol
+		(lib_id "Filter:Choke_Schaffner_RN102-2-02-1M1")
+		(at 93.98 44.45 0)
+		(unit 1)
+		(exclude_from_sim no)
+		(in_bom yes)
+		(on_board yes)
+		(dnp no)
+		(property "Reference" "FL1"
+			(at 93.98 40.386 0)
+			(effects
+				(font
+					(size 1.27 1.27)
+				)
+			)
+		)
+		(property "Value" "Choke_Schaffner_RN102-2-02-1M1"
+			(at 93.472 52.832 0)
+			(effects
+				(font
+					(size 1.27 1.27)
+				)
+			)
+		)
+		(property "Footprint" "Inductor_THT:Choke_Schaffner_RN102-04-14.0x14.0mm"
+			(at 93.98 44.45 0)
+			(effects
+				(font
+					(size 1.27 1.27)
+				)
+				(hide yes)
+			)
+		)
+		(property "Datasheet" "https://www.schaffner.com/products/download/product/datasheet/rn-series-common-mode-chokes-new/"
+			(at 93.98 44.45 0)
+			(effects
+				(font
+					(size 1.27 1.27)
+				)
+				(hide yes)
+			)
+		)
+		(property "Description" "Common mode choke, 2A, 300VAC, 1.1mH, 70mohm, RN-102"
+			(at 93.98 44.45 0)
+			(effects
+				(font
+					(size 1.27 1.27)
+				)
+				(hide yes)
+			)
+		)
+		(pin "2"
+		)
+		(pin "4"
+		)
+		(pin "3"
+		)
+		(pin "1"
+		)
+		(instances
+			(project "STM32_base"
+				(path "/9959bbda-b5da-43e8-8c0f-a51c8fc16f77"
+					(reference "FL1")
 					(unit 1)
 				)
@@
 			(color 0 0 0 0.0000)
 		)
-		(property "Sheetname" "Extra Sheet"
+		(property "Sheetname" "Relay & Mountint Holes"
 			(at 317.5 -0.7116 0)
 			(effects

Commit message: pcb finished, gerber added
Parts:
- removed SW1: SW_Push, Button_Switch_THT:SW_PUSH_6mm, symbol Switch:SW_Push
- added SW1: RST_BTN, Button_Switch_THT:SW_PUSH_6mm, symbol PCM_SL_Devices:Push_Button
Connections:
- net USART_RX is gone; now on net USART1_RX: J2.3 (Pin_3)
- net USART_TX is gone; now on net USART1_TX: J2.2 (Pin_2)
- net GND: now also SW1.1
- net NRST: now also SW1.2
- net Relay_Ctrl: now reaches U1.31 (PA10)
- no-connect marks 28 -> 27
